File: pcb_template/pcb_template.kicad_pcb (KiCad board)
At the start: 2 copper layers, 175 x 100 mm, 8 parts

Commit message: update test,
Parts:
- added FID1: Fiducial, Fiducial:Fiducial_1mm_Mask2mm, F.Cu at (60.5, 51.3)
- added FID2: Fiducial, Fiducial:Fiducial_1mm_Mask2mm, F.Cu at (137.7, 142.2)
- added FID3: Fiducial, Fiducial:Fiducial_1mm_Mask2mm, F.Cu at (184.9, 51.8)
- added FID4: Fiducial, Fiducial:Fiducial_1mm_Mask2mm, F.Cu at (212.3, 92.5)
- added FID5: Fiducial, Fiducial:Fiducial_1mm_Mask2mm, F.Cu at (134.6, 142.2)
- added FID6: Fiducial, Fiducial:Fiducial_1mm_Mask2mm, F.Cu at (209.3, 92.5)
- H1, H2, H3, H4, H5, H6, H7, H8: footprint footprint:MountingHole_3.2mm_M3,rpi_like -> footprint:MountingHole_3.1mm_M3,rpi_like
