File: pcb_template/pcb_template.sch (KiCad schematic (older format))
At the start: 8 parts

Commit message: update test,
Parts:
- added FID1, FID2, FID3, FID4, FID5, FID6: Fiducial, Fiducial:Fiducial_1mm_Mask2mm, symbol Mechanical:Fiducial
- H1, H2, H3, H4, H5, H6, H7, H8: footprint footprint:MountingHole_3.2mm_M3,rpi_like -> footprint:MountingHole_3.1mm_M3,rpi_like
Other:
- moved on the sheet: H1, H2, H3, H4, H5, H6, H7, H8
Changed lines of the file:
@@
 L Mechanical:MountingHole H1
 U 1 1 614714B6
-P 3000 6450
-F 0 "H1" H 3100 6496 50  0000 L CNN
-F 1 "MountingHole" H 3100 6405 50  0000 L CNN
-F 2 "footprint:MountingHole_3.2mm_M3,rpi_like" H 3000 6450 50  0001 C CNN
-F 3 "~" H 3000 6450 50  0001 C CNN
-	1    3000 6450
+P 3600 6700
+F 0 "H1" H 3700 6746 50  0000 L CNN
+F 1 "MountingHole" H 3700 6655 50  0000 L CNN
+F 2 "footprint:MountingHole_3.1mm_M3,rpi_like" H 3600 6700 50  0001 C CNN
+F 3 "~" H 3600 6700 50  0001 C CNN
+	1    3600 6700
 	1    0    0    -1
 $EndComp
@@
 L Mechanical:MountingHole H2
 U 1 1 614716D4
-P 3000 6800
-F 0 "H2" H 3100 6846 50  0000 L CNN
-F 1 "MountingHole" H 3100 6755 50  0000 L CNN
-F 2 "footprint:MountingHole_3.2mm_M3,rpi_like" H 3000 6800 50  0001 C CNN
-F 3 "~" H 3000 6800 50  0001 C CNN
-	1    3000 6800
+P 3600 7000
+F 0 "H2" H 3700 7046 50  0000 L CNN
+F 1 "MountingHole" H 3700 6955 50  0000 L CNN
+F 2 "footprint:MountingHole_3.1mm_M3,rpi_like" H 3600 7000 50  0001 C CNN
+F 3 "~" H 3600 7000 50  0001 C CNN
+	1    3600 7000
 	1    0    0    -1
 $EndComp
@@
 L Mechanical:MountingHole H3
 U 1 1 6147197E
-P 3850 6450
-F 0 "H3" H 3950 6496 50  0000 L CNN
-F 1 "MountingHole" H 3950 6405 50  0000 L CNN
-F 2 "footprint:MountingHole_3.2mm_M3,rpi_like" H 3850 6450 50  0001 C CNN
-F 3 "~" H 3850 6450 50  0001 C CNN
-	1    3850 6450
+P 4500 6700
+F 0 "H3" H 4600 6746 50  0000 L CNN
+F 1 "MountingHole" H 4600 6655 50  0000 L CNN
+F 2 "footprint:MountingHole_3.1mm_M3,rpi_like" H 4500 6700 50  0001 C CNN
+F 3 "~" H 4500 6700 50  0001 C CNN
+	1    4500 6700
 	1    0    0    -1
 $EndComp
@@
 L Mechanical:MountingHole H4
 U 1 1 61471988
-P 3850 6800
-F 0 "H4" H 3950 6846 50  0000 L CNN
-F 1 "MountingHole" H 3950 6755 50  0000 L CNN
-F 2 "footprint:MountingHole_3.2mm_M3,rpi_like" H 3850 6800 50  0001 C CNN
-F 3 "~" H 3850 6800 50  0001 C CNN
-	1    3850 6800
+P 4500 7000
+F 0 "H4" H 4600 7046 50  0000 L CNN
+F 1 "MountingHole" H 4600 6955 50  0000 L CNN
+F 2 "footprint:MountingHole_3.1mm_M3,rpi_like" H 4500 7000 50  0001 C CNN
+F 3 "~" H 4500 7000 50  0001 C CNN
+	1    4500 7000
 	1    0    0    -1
 $EndComp
@@
 L Mechanical:MountingHole H5
 U 1 1 61471D24
-P 4650 6450
-F 0 "H5" H 4750 6496 50  0000 L CNN
-F 1 "MountingHole" H 4750 6405 50  0000 L CNN
-F 2 "footprint:MountingHole_3.2mm_M3,rpi_like" H 4650 6450 50  0001 C CNN
-F 3 "~" H 4650 6450 50  0001 C CNN
-	1    4650 6450
+P 5300 6700
+F 0 "H5" H 5400 6746 50  0000 L CNN
+F 1 "MountingHole" H 5400 6655 50  0000 L CNN
+F 2 "footprint:MountingHole_3.1mm_M3,rpi_like" H 5300 6700 50  0001 C CNN
+F 3 "~" H 5300 6700 50  0001 C CNN
+	1    5300 6700
 	1    0    0    -1
 $EndComp
@@
 L Mechanical:MountingHole H6
 U 1 1 61471D2E
-P 4650 6800
-F 0 "H6" H 4750 6846 50  0000 L CNN
-F 1 "MountingHole" H 4750 6755 50  0000 L CNN
-F 2 "footprint:MountingHole_3.2mm_M3,rpi_like" H 4650 6800 50  0001 C CNN
-F 3 "~" H 4650 6800 50  0001 C CNN
-	1    4650 6800
+P 5300 7000
+F 0 "H6" H 5400 7046 50  0000 L CNN
+F 1 "MountingHole" H 5400 6955 50  0000 L CNN
+F 2 "footprint:MountingHole_3.1mm_M3,rpi_like" H 5300 7000 50  0001 C CNN
+F 3 "~" H 5300 7000 50  0001 C CNN
+	1    5300 7000
 	1    0    0    -1
 $EndComp
@@
 L Mechanical:MountingHole H7
 U 1 1 61471D38
-P 5500 6450
-F 0 "H7" H 5600 6496 50  0000 L CNN
-F 1 "MountingHole" H 5600 6405 50  0000 L CNN
-F 2 "footprint:MountingHole_3.2mm_M3,rpi_like" H 5500 6450 50  0001 C CNN
-F 3 "~" H 5500 6450 50  0001 C CNN
-	1    5500 6450
+P 6200 6700
+F 0 "H7" H 6300 6746 50  0000 L CNN
+F 1 "MountingHole" H 6300 6655 50  0000 L CNN
+F 2 "footprint:MountingHole_3.1mm_M3,rpi_like" H 6200 6700 50  0001 C CNN
+F 3 "~" H 6200 6700 50  0001 C CNN
+	1    6200 6700
 	1    0    0    -1
 $EndComp
@@
 L Mechanical:MountingHole H8
 U 1 1 61471D42
-P 5500 6800
-F 0 "H8" H 5600 6846 50  0000 L CNN
-F 1 "MountingHole" H 5600 6755 50  0000 L CNN
-F 2 "footprint:MountingHole_3.2mm_M3,rpi_like" H 5500 6800 50  0001 C CNN
-F 3 "~" H 5500 6800 50  0001 C CNN
-	1    5500 6800
+P 6200 7000
+F 0 "H8" H 6300 7046 50  0000 L CNN
+F 1 "MountingHole" H 6300 6955 50  0000 L CNN
+F 2 "footprint:MountingHole_3.1mm_M3,rpi_like" H 6200 7000 50  0001 C CNN
+F 3 "~" H 6200 7000 50  0001 C CNN
+	1    6200 7000
 	1    0    0    -1
 $EndComp
+$Comp
+L Mechanical:Fiducial FID3
+U 1 1 61534BDA
+P 2800 6700
+F 0 "FID3" H 2885 6746 50  0000 L CNN
+F 1 "Fiducial" H 2885 6655 50  0000 L CNN
+F 2 "Fiducial:Fiducial_1mm_Mask2mm" H 2800 6700 50  0001 C CNN
+F 3 "~" H 2800 6700 50  0001 C CNN
+	1    2800 6700
+	1    0    0    -1
+$EndComp
+$Comp
+L Mechanical:Fiducial FID1
+U 1 1 6153927D
+P 2100 6700
+F 0 "FID1" H 2185 6746 50  0000 L CNN
+F 1 "Fiducial" H 2185 6655 50  0000 L CNN
+F 2 "Fiducial:Fiducial_1mm_Mask2mm" H 2100 6700 50  0001 C CNN
+F 3 "~" H 2100 6700 50  0001 C CNN
+	1    2100 6700
+	1    0    0    -1
+$EndComp
+$Comp
+L Mechanical:Fiducial FID2
+U 1 1 615392CF
+P 2100 7000
+F 0 "FID2" H 2185 7046 50  0000 L CNN
+F 1 "Fiducial" H 2185 6955 50  0000 L CNN
+F 2 "Fiducial:Fiducial_1mm_Mask2mm" H 2100 7000 50  0001 C CNN
+F 3 "~" H 2100 7000 50  0001 C CNN
+	1    2100 7000
+	1    0    0    -1
+$EndComp
+$Comp
+L Mechanical:Fiducial FID4
+U 1 1 61538E26
+P 2800 7000
+F 0 "FID4" H 2885 7046 50  0000 L CNN
+F 1 "Fiducial" H 2885 6955 50  0000 L CNN
+F 2 "Fiducial:Fiducial_1mm_Mask2mm" H 2800 7000 50  0001 C CNN
+F 3 "~" H 2800 7000 50  0001 C CNN
+	1    2800 7000
+	1    0    0    -1
+$EndComp
+$Comp
+L Mechanical:Fiducial FID5
+U 1 1 615355C5
+P 2100 7300
+F 0 "FID5" H 2185 7346 50  0000 L CNN
+F 1 "Fiducial" H 2185 7255 50  0000 L CNN
+F 2 "Fiducial:Fiducial_1mm_Mask2mm" H 2100 7300 50  0001 C CNN
+F 3 "~" H 2100 7300 50  0001 C CNN
+	1    2100 7300
+	1    0    0    -1
+$EndComp
+$Comp
+L Mechanical:Fiducial FID6
+U 1 1 61535617
+P 2800 7300
+F 0 "FID6" H 2885 7346 50  0000 L CNN
+F 1 "Fiducial" H 2885 7255 50  0000 L CNN
+F 2 "Fiducial:Fiducial_1mm_Mask2mm" H 2800 7300 50  0001 C CNN
+F 3 "~" H 2800 7300 50  0001 C CNN
+	1    2800 7300
+	1    0    0    -1
+$EndComp
